File: stone.kicad_pcb (KiCad board)
At the start: 4 copper layers, 18 x 26 mm, 43 parts, among them J1 Conn_ARM_SWD_TagConnect_TC203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, J2 UHF_ANT, J3 GNSS_ANT, Q1 AO3400A, Q4 DMC2710UV-7, U1 STM32C011F4Ux, U2 LIS2DH, U3 LP5912-3.3DRV, U4 MAX-M10S, U5 E22-400MM22S

Commit message: added reverse voltage p fet
Parts:
- removed D5: 1N5819WS, Diode_SMD:D_SOD-323
- added Q2: AO3401A, Package_TO_SOT_SMD:SOT-23, B.Cu at (136.7, 51.5)
- moved R1 3.12 mm to (135.1, 54.5), turned to -90 degrees
- moved BT1 2.27 mm to (137.2, 54.0), turned to -90 degrees
- moved R2 1.28 mm to (135.1, 56.5)
- moved C1 0.80 mm to (136.9, 49.0)
Routing:
- net VBAT: track 7.01 -> 4.78 mm
- net VIN: track 3.49 -> 4.93 mm
- net /VBAT_SNS: track 12.7 -> 11.3 mm
- net +3V3: track 19.1 -> 19.8 mm
- net /SWDIO: track 15.5 -> 16.2 mm
- net GND: vias 30 -> 27

Commit message: updated silk
Other:
- board text added: "+"
- board text added: "-"
- board text added: "3.4-6.5V"
- board text added: "UCSC"
- board text removed: "6.5V MAX!"
Changed lines of the file:
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@@
 			(at 0 2.4 0)
 			(layer "B.SilkS")
+			(hide yes)
 			(effects
 				(font
@@
 		)
 	)
-	(gr_text "6.5V MAX!"
-		(at 138.684 52.8828 90)
+	(gr_text "3.4-6.5V"
+		(at 134.62 40.894 90)
+		(layer "B.SilkS")
+		(effects
+			(font
+				(size 0.762 0.762)
+				(bold yes)
+			)
+			(justify left bottom mirror)
+		)
+	)
+	(gr_text "UCSC"
+		(at 137.414 43.434 90)
+		(layer "B.SilkS")
+		(effects
+			(font
+				(size 0.762 0.762)
+				(bold yes)
+			)
+			(justify left bottom mirror)
+		)
+	)
+	(gr_text "+"
+		(at 138.684 52.197 90)
+		(layer "B.SilkS")
+		(effects
+			(font
+				(size 0.762 0.762)
+				(bold yes)
+			)
+			(justify left bottom mirror)
+		)
+	)
+	(gr_text "-"
+		(at 138.684 57.023 90)
 		(layer "B.SilkS")
 		(effects
@@
 	)
 	(segment
-		(start 138.1711 50.772)
-		(end 137.8455 50.772)
-		(width 0.3556)
-		(layer "F.Cu")
-		(net "VIN")
-	)
-	(segment
-		(start 137.8455 50.772)
-		(end 137.3426 50.772)
+		(start 138.1711 50.6681)
+		(end 138.049 50.546)
 		(width 0.3556)
 		(layer "F.Cu")
@@
 	)
 	(segment
-		(start 137.3426 50.772)
-		(end 137.2586 50.688)
-		(width 0.3556)
-		(layer "F.Cu")
-		(net "VIN")
-	)
-	(segment
 		(start 137.2586 49.388)
 		(end 137.333586 49.388)
@@
 	)
 	(segment
-		(start 138.0744 50.772)
-		(end 137.8712 50.772)
+		(start 138.049 50.546)
+		(end 137.668 50.546)
+		(width 0.3556)
+		(layer "F.Cu")
+		(net "VIN")
+	)
+	(segment
+		(start 138.1711 50.772)
+		(end 138.1711 50.6681)
+		(width 0.3556)
+		(layer "F.Cu")
+		(net "VIN")
+	)
+	(segment
+		(start 137.4006 50.546)
+		(end 137.2586 50.688)
+		(width 0.3556)
+		(layer "F.Cu")
+		(net "VIN")
+	)
+	(segment
+		(start 137.668 50.546)
+		(end 137.4006 50.546)
 		(width 0.3556)
 		(layer "F.Cu")
@@
 	)
 	(via
-		(at 137.6423 50.772)
+		(at 137.668 50.546)
 		(size 0.3556)
 		(drill 0.2032)
@@
 	)
 	(segment
-		(start 135.7145 50.551)
-		(end 137.663 50.551)
-		(width 0.3556)
-		(layer "B.Cu")
-		(net "VIN")
-	)
-	(segment
-		(start 137.668 50.7463)
-		(end 137.6423 50.772)
-		(width 0.3556)
-		(layer "B.Cu")
-		(net "VIN")
-	)
-	(segment
-		(start 137.6423 50.772)
-		(end 137.6423 49.696714)
-		(width 0.3556)
-		(layer "B.Cu")
-		(net "VIN")
-	)
-	(segment
 		(start 137.6423 49.696714)
 		(end 137.582512 49.636926)
@@
 	)
 	(segment
+		(start 137.668 50.546)
+		(end 137.6423 50.5203)
+		(width 0.3556)
+		(layer "B.Cu")
+		(net "VIN")
+	)
+	(segment
 		(start 137.663 50.551)
-		(end 137.668 50.546)
+		(end 135.7145 50.551)
 		(width 0.3556)
 		(layer "B.Cu")
@@
 	(segment
 		(start 137.668 50.546)
-		(end 137.668 50.7463)
-		(width 0.3556)
-		(layer "B.Cu")
+		(end 137.663 50.551)
+		(width 0.3556)
+		(layer "B.Cu")
+		(net "VIN")
+	)
+	(segment
+		(start 137.6423 50.5203)
+		(end 137.6423 49.696714)
+		(width 0.3556)
+		(layer "B.Cu")
